Commit message: 修改bottom_joint相关，解决报错前保存

File: src/marm_description/urdf/arm.xacro (robot description, xacro)
@@ -63,5 +63,5 @@
                        <box size="1 1 0.02" />
                   </geometry>
-              <material name="Brown" />
+              <material name="Black" />
         </visual>
         <collision>

Commit message: 通过添加dummy_link解决了警告问题，但是这样模型地板还是在地下，需解决

File: src/marm_description/urdf/arm.xacro (robot description, xacro)
@@ -74,4 +74,5 @@
     </link>
     <!-- /////////////////////////////////////   BASE LINK    ////////////////////////////////////////////// -->
+    <link name="dummy_link"></link>
     <link name="base_link">
         <visual>
@@ -90,4 +91,8 @@
         <xacro:inertial_matrix mass="1"/>
     </link>
+    <joint name="dummy_joint" type="fixed">
+     <parent link="dummy_link"/>
+     <child link="base_link"/>
+   </joint>
     <joint name="joint1" type="revolute">
         <parent link="base_link"/>
